File: pcb/pcb_2layer.kicad_pcb (KiCad board)
At the start: 2 copper layers, 71.5 x 115.4 mm, 163 parts, among them J1 AudioJack3_SwitchTR, J100 Conn_02x05_Odd_Even, J102 Conn_01x03, J500 FPC_18P_1.0MM, J600 USB_B_Micro, Q300 IRLML6402, SW1 SW_SP3T, SW700 SW_Push, SW701 SW_Push, SW702 SW_Push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

Commit message: pcb: rev 0.1
Routing:
- net GND: track 129.2 -> 104.9 mm, vias 195 -> 185
- added copper zone on In1.Cu, net +3V3
- added copper zone on In1.Cu, net GND
- added copper zone on In2.Cu, net GND
- added copper zone on In1.Cu, net Net-(C20-Pad1)
Other:
- copper layers 2 -> 4
