File: pcb/cpu.sch (KiCad schematic (older format))
At the start: 28 parts, among them J100 Conn_02x05_Odd_Even, J101 Conn_02x05_Odd_Even, J102 Conn_01x03, U100 MCIMX7S5EVM08SC, Y100 24MHz, Y101 32.768kHz

Commit message: pcb: adding lpc5500
Parts:
- removed J101: Conn_02x05_Odd_Even, Connector_PinHeader_1.27mm:PinHeader_2x05_P1.27mm_Vertical_SMD, symbol Connector_Generic:Conn_02x05_Odd_Even
- removed R104, R107: 10K-DNP, Resistor_SMD:R_0603_1608Metric, symbol Device:R
- removed R105, R106: 10K, Resistor_SMD:R_0603_1608Metric, symbol Device:R
- removed RN100, RN101, RN102: 10K, Resistor_SMD:R_Array_Convex_4x0402, symbol Device:R_Pack04
- removed U100: MCIMX7S5EVM08SC, footprints:BGA-541_25x25_19.0x19.0mm, symbol symbols:MCIMX7S5EVM08SC
- added U?: LPC5500, Package_QFP:TQFP-100-1EP_14x14mm_P0.5mm_EP5x5mm_ThermalVias, symbol symbols:LPC5500
Connections:
- net labels removed: +RTC, BT_CFG_1, BT_CFG_10, BT_CFG_11, BT_CFG_12, BT_CFG_13, BT_CFG_14, BT_CFG_2, BT_CFG_3, BT_CFG_4, BT_CFG_5, BT_CFG_6, CPLD_JTAG_TCK, CPLD_JTAG_TDI, CPLD_JTAG_TDO, CPLD_JTAG_TMS
- wire segments 143 -> 95
- no-connect marks 14 -> 1
Other:
- note removed: "BOOTMODE[1:0]:\n00 - Boot from fuses\n01 - Serial Downloader\n10 - Internal Boot\n11 - Reserved"
- note removed: "CPLD JTAG"
- moved on the sheet: C101, C102, C103, C104, R102, R103, Y100, Y101

Commit message: pcb: move cpu power to power page
Parts:
- removed C101, C102: 18pF-DNP, Capacitor_SMD:C_0402_1005Metric, symbol Device:C
- removed C103, C104: 18pF, Capacitor_SMD:C_0402_1005Metric, symbol Device:C
- removed R102: 1M, Resistor_SMD:R_0603_1608Metric, symbol Device:R
- removed R103: 4.75M-DNP, Resistor_SMD:R_0603_1608Metric, symbol Device:R
- removed U?: LPC5500, Package_QFP:TQFP-100-1EP_14x14mm_P0.5mm_EP5x5mm_ThermalVias, symbol symbols:LPC5500
- removed Y100: 24MHz, Oscillator:Oscillator_SMD_Abracon_ASE-4Pin_3.2x2.5mm, symbol Device:Crystal_GND24
- removed Y101: 32.768kHz, Crystal:Crystal_SMD_TXC_9HT11-2Pin_2.0x1.2mm_HandSoldering, symbol Device:Crystal
Connections:
- wire segments 95 -> 59
Other:
- note removed: "There are already lot of decoupling\ncaps just next to it."
- moved on the sheet: C100

Commit message: pcb: rev 0.1
Parts:
- removed C100, C107, C108: 220nF, Capacitor_SMD:C_0402_1005Metric, symbol Device:C
- removed C110: 2.2uF, Capacitor_SMD:C_0402_1005Metric, symbol Device:C
- removed R109: 10K, Resistor_SMD:R_0603_1608Metric, symbol Device:R
- added D101: LED, LED_THT:LED_D5.0mm, symbol Device:LED
- added R100: 1K, Resistor_SMD:R_0603_1608Metric, symbol Device:R
- added U100: LPC5500, Package_QFP:TQFP-100-1EP_14x14mm_P0.5mm_EP5x5mm_ThermalVias, symbol symbols:LPC5500
Connections:
- net labels added: ADC1_IN0, FC0_USART_RXD, FC0_USART_TXD, HOLD, LED, SAI1_MCLK, SAI1_TXC, SAI1_TXD, SAI1_TXFS, SD0_CLK, SD0_CMD, SD0_D0, SD0_D1, SD0_D2, SD0_D3, STN_CP, STN_CPG, STN_CPL, STN_D0, STN_D1, STN_FR, STN_S, STN_ST, SW_A, SW_B, SW_DN, SW_LE, SW_RI, SW_SE, SW_ST, SW_UP, ~LCD_PWR_EN, ~SD0_CD, ~SD0_PWR_EN
- net labels removed: +1V8A, MPU_JTAG_TDI, MPU_JTAG_TRST, PMIC_STBY_REQ, UART3_CTS, UART3_RTS, UART3_RXD, UART3_TXD
- wire segments 59 -> 68
- no-connect marks 1 -> 2
Other:
- note added: "To Audio DAC\n"
- note removed: "To WiFi & BT"
- moved on the sheet: J102, R110, R111

Commit message: pcb: fixing voltage domain
Connections:
- net labels added: +1V8
- wire segments 68 -> 69
Changed lines of the file:
@@
 Text GLabel 4200 3500 2    50   Input ~ 0
 ~SD0_CD
-Connection ~ 4500 1400
 Wire Wire Line
 	4900 1400 4500 1400
-$Comp
-L power:+3V3 #PWR?
-U 1 1 5DA800C1
-P 4500 1400
-AR Path="/5DB2122B/5DA800C1" Ref="#PWR?"  Part="1"
-AR Path="/5D180A01/5DA800C1" Ref="#PWR0123"  Part="1"
-F 0 "#PWR0123" H 4500 1250 50  0001 C CNN
-F 1 "+3V3" H 4515 1573 50  0000 C CNN
-F 2 "" H 4500 1400 50  0001 C CNN
-F 3 "" H 4500 1400 50  0001 C CNN
-	1    4500 1400
-	1    0    0    -1
-$EndComp
 $Comp
 L Device:R R111
@@
 Wire Wire Line
 	4900 5950 5100 5950
+$Comp
+L power:+1V8 #PWR?
+U 1 1 5D8B4E32
+P 4500 1300
+F 0 "#PWR?" H 4500 1150 50  0001 C CNN
+F 1 "+1V8" H 4515 1473 50  0000 C CNN
+F 2 "" H 4500 1300 50  0001 C CNN
+F 3 "" H 4500 1300 50  0001 C CNN
+	1    4500 1300
+	1    0    0    -1
+$EndComp
+Wire Wire Line
+	4500 1300 4500 1400
+Connection ~ 4500 1400
 $EndSCHEMATC

Commit message: pcb: fixing i2c numbering; add filtering for lcd
Connections:
- net labels removed: +1V8
- wire segments 69 -> 68
Changed lines of the file:
@@
 Wire Wire Line
 	4500 3100 5100 3100
-Text GLabel 5100 3200 2    50   BiDi ~ 0
+Text GLabel 5100 3100 2    50   BiDi ~ 0
 I2C1_SDA
-Text GLabel 5100 3100 2    50   Output ~ 0
+Text GLabel 5100 3200 2    50   Output ~ 0
 I2C1_SCL
 Wire Wire Line
@@
 	4900 5950 5100 5950
 $Comp
-L power:+1V8 #PWR?
-U 1 1 5D8B4E32
-P 4500 1300
-F 0 "#PWR?" H 4500 1150 50  0001 C CNN
-F 1 "+1V8" H 4515 1473 50  0000 C CNN
-F 2 "" H 4500 1300 50  0001 C CNN
-F 3 "" H 4500 1300 50  0001 C CNN
-	1    4500 1300
+L power:+3V3 #PWR0106
+U 1 1 5DB9934B
+P 4500 1400
+F 0 "#PWR0106" H 4500 1250 50  0001 C CNN
+F 1 "+3V3" H 4515 1573 50  0000 C CNN
+F 2 "" H 4500 1400 50  0001 C CNN
+F 3 "" H 4500 1400 50  0001 C CNN
+	1    4500 1400
 	1    0    0    -1
 $EndComp
-Wire Wire Line
-	4500 1300 4500 1400
 Connection ~ 4500 1400
 $EndSCHEMATC

Commit message: pcb: use crystal instead
Connections:
- net labels added: CODEC_RST
- wire segments 68 -> 69
Changed lines of the file:
@@
 	6500 2900 6700 2900
 Wire Wire Line
-	6700 2200 6500 2200
+	6700 2700 6500 2700
+Wire Wire Line
+	6700 2500 6500 2500
+Wire Wire Line
+	4200 1900 4000 1900
+Wire Wire Line
+	6700 2400 6500 2400
+Wire Wire Line
+	6700 3800 6500 3800
+Wire Wire Line
+	6700 4200 6500 4200
 Wire Wire Line
 	6700 3100 6500 3100
 Wire Wire Line
-	6700 4200 6500 4200
-Wire Wire Line
-	6700 3800 6500 3800
-Wire Wire Line
-	6700 2400 6500 2400
-Wire Wire Line
-	4200 1900 4000 1900
-Wire Wire Line
-	6700 2500 6500 2500
-Wire Wire Line
-	6700 2700 6500 2700
+	6700 2200 6500 2200
+Text GLabel 6700 2700 2    50   Output ~ 0
+STN_S
+Text GLabel 6700 2500 2    50   Output ~ 0
+STN_FR
+Text GLabel 4200 1900 2    50   Output ~ 0
+STN_CP
+Text GLabel 6700 2400 2    50   Output ~ 0
+STN_D1
+Text GLabel 6700 3800 2    50   Output ~ 0
+STN_D0
+Text GLabel 6700 4200 2    50   Output ~ 0
+STN_ST
+Text GLabel 6700 3100 2    50   Output ~ 0
+STN_CPL
 Text GLabel 6700 2200 2    50   Output ~ 0
-STN_S
-Text GLabel 6700 3100 2    50   Output ~ 0
-STN_FR
-Text GLabel 6700 4200 2    50   Output ~ 0
-STN_CP
-Text GLabel 6700 3800 2    50   Output ~ 0
-STN_D1
-Text GLabel 6700 2400 2    50   Output ~ 0
-STN_D0
-Text GLabel 4200 1900 2    50   Output ~ 0
-STN_ST
-Text GLabel 6700 2500 2    50   Output ~ 0
-STN_CPL
-Text GLabel 6700 2700 2    50   Output ~ 0
 STN_CPG
 Text GLabel 4200 4600 2    50   Input ~ 0
@@
 $EndComp
 Connection ~ 4500 1400
+Text GLabel 6700 4600 2    50   Output ~ 0
+CODEC_RST
+Wire Wire Line
+	6500 4600 6700 4600
 $EndSCHEMATC
